File: dash/PCB/_autosave-bargraph.kicad_pcb (KiCad board)
At the start: 2 copper layers, 100 x 59.1 mm, 100 parts, among them IC1 ATMEGA328-P, J1 DB9, P1 USB_OTG, P2 CONN_02X05, P3 CONN_02X05, P4 CONN_02X05, P5 CONN_02X05, Q1 BC557, Q2 BC547, U1 CH340G, U2 7805, U3 arduino_mini, U4 74HC4094, U5 74HC4094, U6 74HC4094, U7 74HC4094, X1 CRYSTAL_SMD, X2 CRYSTAL_SMD

Commit message: Fixing bugs in the PCB designe
Parts:
- removed P2, P3, P4, P5: CONN_02X05, Pin_Headers:Pin_Header_Straight_2x05
- removed U3: arduino_mini, addlol:arduino_nano
- added P2a1: CONN_02X05, Pin_Headers:Pin_Header_Straight_2x05, F.Cu at (87.0, 100.2)
- added P2b1: CONN_02X05, Pin_Headers:Pin_Header_Straight_2x05, F.Cu at (87.0, 81.3)
- added P3a1: CONN_02X05, Pin_Headers:Pin_Header_Straight_2x05, F.Cu at (147.4, 101.6)
- added P3b1: CONN_02X05, Pin_Headers:Pin_Header_Straight_2x05, F.Cu at (148.1, 80.7)
- added R49: 1k, Resistors_SMD:R_0805_HandSoldering, B.Cu at (94.7, 106.1)
- added R50: 1kR, Resistors_SMD:R_0805_HandSoldering, B.Cu at (97.2, 106.1)
- added R51: R, Resistors_SMD:R_0805_HandSoldering, B.Cu at (84.0, 106.1)
- added R52: 1k, Resistors_SMD:R_0805_HandSoldering, B.Cu at (89.6, 106.1)
- added R53: 1k, Resistors_SMD:R_0805_HandSoldering, B.Cu at (92.1, 106.1)
- AFF1: value LTS-6980HR -> 7SEGMENTS
- C1, C10, C11, C12, C13, C2, C3, C4, C5, C6, C7, C8, C9, D1, D10, D11, D12, D2, D3, D4, D5, D6, D7, D8, D9, IC1, R1, R10, R11, R12, R2, R3, R38, R4, R40, R45, R5, R7, R8, R9, X1, X2: moved to B.Cu
- J1: footprint Connect:DB9FC -> Pin_Headers:Pin_Header_Straight_2x05
- Q2: moved to F.Cu
- U2: value 7805 -> LM7805CT; footprint TO_SOT_Packages_THT:TO-220_Neutral123_Horizontal -> TO_SOT_Packages_THT:TO-220_Neutral123_Horizontal_LargePads
- moved X1 163.2 mm to (68.1, 138.9), turned to 270 degrees
- moved R9 157.5 mm to (79.8, 130.5)
- moved C6 155.7 mm to (71.2, 130.0), turned to 180 degrees
- moved C1 138.5 mm to (231.1, 121.7), turned to 0 degrees
- moved C12 129.7 mm to (231.1, 123.7), turned to 0 degrees
- moved D1 119.8 mm to (167.7, 139.6)
- moved C8 111.1 mm to (231.1, 119.7), turned to 0 degrees
- moved D2 110.3 mm to (113.3, 140.1)
- moved Q2 107.9 mm to (138.1, 102.7)
- moved D7 103.8 mm to (122.5, 140.2), turned to 270 degrees
- moved R45 99.1 mm to (131.9, 100.0), turned to 180 degrees
- moved D5 92.1 mm to (109.0, 125.1), turned to 270 degrees
- moved R40 83.8 mm to (150.0, 106.1), turned to 0 degrees
- moved Q1 83.7 mm to (151.6, 108.8), turned to 180 degrees
- moved C13 83.7 mm to (159.3, 58.6), turned to 0 degrees
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Connections:
- AFF1 pad 3: GNDREF -> /Vcc
- AFF1 pad 8: GNDREF -> /Vcc
- H1 pad 9: /D12 -> Net-(H1-Pad9)
- J1 pad 6: /12Vraw -> /oilP
- J1 pad 7: /oilP -> Net-(J1-Pad7)
- J1 pad 9: Net-(J1-Pad9) -> /12Vraw
- U2 pad 1: GNDREF -> Net-(C4-Pad1)
- U2 pad 2: /Vcc -> GNDREF
- U2 pad 3: Net-(C4-Pad1) -> /Vcc
- X1 pad 2: Net-(U1-Pad10) -> GNDREF
- X1 pad 3: GNDREF -> Net-(U1-Pad10)
- X2 pad 1: Net-(IC1-Pad8) -> Net-(IC1-Pad7)
- X2 pad 2: Net-(IC1-Pad7) -> GNDREF
- X2 pad 3: GNDREF -> Net-(IC1-Pad8)
Routing:
- net GNDREF: track 297.0 -> 618.3 mm, vias 4 -> 6
- net /Vcc: track 106.5 -> 382.3 mm, vias 0 -> 7
- net /gearDown: track 0.00 -> 82.5 mm, vias 0 -> 2
- net /gearUp: track 0.00 -> 78.7 mm
- net /oilP: track 0.00 -> 78.3 mm
- net /D2: track 0.00 -> 78.0 mm, vias 0 -> 2
- net /D3: track 0.00 -> 69.8 mm, vias 0 -> 2
- net /D11: track 0.00 -> 68.5 mm
- net /D12: track 0.00 -> 66.2 mm, vias 0 -> 2
- net /neutral: track 0.00 -> 62.0 mm
- net /A0: track 0.00 -> 43.7 mm
- net /rpm: track 0.00 -> 42.6 mm, vias 0 -> 1
- net /A6: track 0.00 -> 42.4 mm, vias 0 -> 2
- net /D10: track 0.00 -> 34.6 mm
- net Net-(D10-Pad1): track 0.00 -> 34.3 mm, vias 0 -> 6
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Other:
- net class 0.3 added: clearance 0.2, trace_width 0.3, via_dia 1.5, via_drill 0.8
- net class 0.4 added: clearance 0.2, trace_width 0.4, via_dia 1.5, via_drill 0.8
- net class 0.5 added: clearance 0.2, trace_width 0.5, via_dia 1.5, via_drill 0.8
- net class Default: trace_width 0.25 -> 0.3
- net class extra width removed
- board text added: "."
- board text added: "HVR2 2016"

Commit message: adding stuff
Parts:
- removed C12, C8: 100n, Capacitors_SMD:C_0805_HandSoldering
- removed P2a1, P2b1, P3a1, P3b1: CONN_02X05, Pin_Headers:Pin_Header_Straight_2x05
- added P2: CONN_01X05, Socket_Strips:Socket_Strip_Straight_1x05, B.Cu at (85.1, 98.5)
- added P3: CONN_01X05, Pin_Headers:Pin_Header_Straight_1x05, B.Cu at (85.1, 80.6)
- added P4: CONN_01X05, Socket_Strips:Socket_Strip_Straight_1x05, B.Cu at (144.8, 98.4)
- added P5: CONN_01X05, Pin_Headers:Pin_Header_Straight_1x05, B.Cu at (144.8, 80.6)
- added P6: CONN_01X02, Socket_Strips:Socket_Strip_Straight_1x02, F.Cu at (169.5, 107.9)
- C1, J1, R38, R45: moved to F.Cu
- C6: value C -> 100n
- Q1, Q2: moved to B.Cu
- R13, R14, R15, R16, R17, R18, R19, R20, R21, R22, R23, R24, R25, R26, R27, R28, R29, R30, R31, R32, R33, R34, R35, R36, R37, R39, R41, R42, R43, R44, R46, R47: value 560 -> 330
- moved C1 167.3 mm to (77.0, 56.6), turned to 270 degrees
- moved X1 14.4 mm to (82.2, 135.8)
- moved R14 9.99 mm to (92.5, 39.4)
- moved R16 9.99 mm to (97.5, 39.4)
- moved R18 9.99 mm to (102.6, 39.4)
- moved R19 9.99 mm to (105.2, 39.4)
- moved R21 9.99 mm to (110.2, 39.4)
- moved R13 9.99 mm to (89.9, 39.4)
- moved R15 9.99 mm to (95.0, 39.4)
- moved R17 9.99 mm to (100.1, 39.4)
- moved R20 9.99 mm to (107.7, 39.4)
- moved R22 9.99 mm to (112.8, 39.4)
- moved bar_green1 9.91 mm to (89.8, 43.1)
- moved R8 9.38 mm to (73.8, 125.3), turned to 315 degrees
- moved R45 7.61 mm to (124.3, 99.6)
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Connections:
- AFF1 pad 3: /Vcc -> Net-(AFF1-Pad3)
- D13 pad 2: /12vraw -> /12vF
- D3 pad 2: Net-(D3-Pad2) -> /12vF
- H1 pad 7: /A6 -> Net-(H1-Pad7)
- IC1 pad 19: /A6 -> Net-(IC1-Pad19)
- J1 pad 2: /gearUp -> /gearDown
- J1 pad 3: /gearDown -> /neutral
- J1 pad 4: /neutral -> /gearUp
- J1 pad 5: GNDREF -> Net-(J1-Pad5)
- J1 pad 6: /oilP -> Net-(J1-Pad6)
- J1 pad 7: Net-(J1-Pad7) -> GNDREF
- J1 pad 8: /extShiftLight -> GNDREF
- J1 pad 9: /12Vraw -> /12vraw
- Q1 pad 3: /12vraw -> /12vF
- R3 pad 1: Net-(D3-Pad2) -> /12vF
- R3 pad 2: /12Vraw -> /12vraw
- U1 pad 1: /Vcc -> GNDREF
- U1 pad 11: Net-(P1-Pad2) -> Net-(U1-Pad11)
- U1 pad 12: Net-(P1-Pad3) -> Net-(U1-Pad12)
- U1 pad 13: Net-(C6-Pad1) -> /DTR
- U1 pad 14: /tx -> Net-(U1-Pad14)
- U1 pad 15: /rx -> Net-(U1-Pad15)
- U1 pad 16: GNDREF -> /Vcc
- U1 pad 4: /DTR -> Net-(C6-Pad1)
- U1 pad 5: Net-(U1-Pad5) -> Net-(P1-Pad3)
- U1 pad 6: Net-(U1-Pad6) -> Net-(P1-Pad2)
- X1 pad 1: Net-(U1-Pad9) -> Net-(U1-Pad8)
- X1 pad 3: Net-(U1-Pad10) -> Net-(U1-Pad7)
Routing:
- net /12vF: track 0.00 -> 160.5 mm, vias 0 -> 2
- net GNDREF: track 618.3 -> 744.7 mm, vias 6 -> 7
- net /12vraw: track 121.0 -> 9.34 mm, vias 0 -> 1
- net /Vcc: track 382.3 -> 454.7 mm, vias 7 -> 9
- net /A6: track 42.4 -> 0.00 mm, vias 2 -> 0
- net /oilP: track 78.3 -> 47.8 mm
- net /U2_1: track 21.2 -> 38.8 mm
- net /U2_5: track 23.6 -> 40.3 mm
- net /extShiftLight: track 27.2 -> 11.3 mm, vias 2 -> 0
- net (no net): track 0.13 -> 15.8 mm, vias 0 -> 6
- net /intShiftLight: track 156.1 -> 140.9 mm, vias 0 -> 2
- net /U2_0: track 18.2 -> 31.9 mm
- net /RST: track 32.6 -> 19.4 mm
- net /U2_4: track 20.9 -> 33.9 mm
- net /U1_7: track 22.4 -> 34.1 mm
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Other:
- board size 100 x 59.1 mm -> 120 x 127 mm
- board text added: "+"
- board text added: "D4 D5 D6 D7 D8"
- board text added: "Gnd NC A7 NC A5 A4 A3 A2 A1 Vcc"
- board text added: "Vcc 12V Shft Gnd Gnd"
- board text added: "gearD gearU NC Gnd NC"
- board text added: "rpm neut NC Gnd 12V"
- board text added: "v0.2"
- board text added: "|"
