File: dash/PCB/bargraph.sch (KiCad schematic (older format))
At the start: 69 parts, among them IC1 ATMEGA328-P, P1 USB_OTG, U1 7805, U2 CH340G, Y1 12MHz

Commit message: progress
Parts:
- removed C? (x2): C, symbol C
- removed C?: 1n, symbol C
- removed D?: 1n4007, symbol D
- removed Y1: 12MHz, symbol Crystal_Small
- added C10: 100n, Capacitors_SMD:C_0805_HandSoldering, symbol C
- added C4, C5: CP1, symbol CP1
- added D13, D14, D15, D16, D17: LED, symbol LED
- added D3: D_Schottky_Small, symbol D_Schottky_Small
- added D5, D6, D7, D8: 5.1V, Diodes_SMD:MELF_Handsoldering, symbol ZENER
- added H1: pin_header_10, symbol pin_header_10
- added Q1: BC557, TO-92, symbol BC557
- added Q2: BC547, TO-92, symbol BC547
- added R38: 1R, Resistors_SMD:R_0805_HandSoldering, symbol R
- added R4, R5, R6, R7: 2k2, Resistors_SMD:R_0805_HandSoldering, symbol R
- added R40: 10k, Resistors_SMD:R_0805_HandSoldering, symbol R
- added R45: 3k3, Resistors_SMD:R_0805_HandSoldering, symbol R
- added R48: 100R, Resistors_SMD:R_0805_HandSoldering, symbol R
- added R8: 1kR, Resistors_SMD:R_0805_HandSoldering, symbol R
- added U3: arduino_mini, DIL20, symbol arduino_mini
- added X1, X2: CRYSTAL_SMD, SMD_Packages:Ceramic_Filter, symbol CRYSTAL_SMD
- C1: footprint (none) -> Capacitors_SMD:C_0805_HandSoldering
- C11, C12, C13, C2, C3, C7, C8, C9: renamed from C?; footprint (none) -> Capacitors_SMD:C_0805_HandSoldering
- C6: renamed from C4; footprint (none) -> Capacitors_SMD:C_0805_HandSoldering
- D1, D10, D11, D12, D2, D4, D9: renamed from D?; footprint (none) -> Diodes_SMD:MELF_Handsoldering
- R1, R10, R11, R12, R13, R14, R15, R16, R17, R18, R19, R2, R20, R21, R22, R23, R24, R25, R26, R27, R28, R29, R3, R30, R31, R32, R33, R34, R35, R36, R37, R39, R41, R42, R43, R44, R46, R47, R9: renamed from R?; footprint (none) -> Resistors_SMD:R_0805_HandSoldering
- U1: renamed from U2; footprint (none) -> Housings_SOIC:SOIC-16_3.9x9.9mm_Pitch1.27mm
- U2: renamed from U1; footprint s -> TO_SOT_Packages_THT:TO-220_Neutral123_Horizontal
- gave numbers to parts that had none: 1
Connections:
- net labels added: 12vraw, D0, D1, D2, D3, D4, D5, D6, DTR, RST, extShiftLight
- wire segments 139 -> 169
- no-connect marks 6 -> 14
Other:
- moved on the sheet: C1, C6, D1, P1, R12, R3, R9, U1, bar_green1, bar_red1, bar_ylw1

Commit message: One of the boards completed at least
Parts:
- removed C4: CP1, symbol CP1
- removed D16: LED, symbol LED
- added C4: 470n, Capacitors_SMD:C_0805_HandSoldering, symbol C
- added J1: DB9, Connect:DB9FC, symbol DB9
- added P2, P3, P4, P5: CONN_02X05, Pin_Headers:Pin_Header_Straight_2x05, symbol CONN_02X05
- added U4, U5, U6, U7: 74HC4094, Housings_DIP:DIP-16_W7.62mm, symbol 74HC4094
- AFF1: footprint (none) -> addlol:7seg
- C5: value CP1 -> 100u; footprint (none) -> Capacitors_SMD:c_elec_6.3x5.8
- D13, D14, D15, D17: footprint (none) -> LEDs:LED-5MM
- D3: footprint (none) -> Diodes_SMD:SOD-123
- H1: footprint (none) -> Pin_Headers:Pin_Header_Straight_1x10
- P1: footprint (none) -> Connect:USB_Micro-B_10103594-0001LF
- Q1, Q2: footprint TO-92 -> TO_SOT_Packages_THT:TO-92_Inline_Wide
- R45: value 3k3 -> 2k7
- R48: value 100R -> 60R
- U3: footprint DIL20 -> addlol:arduino_nano
- X1, X2: footprint SMD_Packages:Ceramic_Filter -> addlol:cer_res
Connections:
- net labels added: intShiftLight
- net labels removed: 74HC4094, d6, vcc
- wire segments 169 -> 187
- no-connect marks 14 -> 25
Other:
- moved on the sheet: D13, D14, D15, D17, Q1, Q2, R13, R14, R15, R16, R17, R18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

Commit message: Fixing bugs in the PCB designe
Parts:
- removed AFF1: LTS-6980HR, addlol:7seg, symbol LTS-6980HR
- removed U2: 7805, TO_SOT_Packages_THT:TO-220_Neutral123_Horizontal, symbol AP1117
- added AFF1: 7SEGMENTS, addlol:7seg, symbol 7SEGMENTS
- added R49, R52, R53: 1k, Resistors_SMD:R_0805_HandSoldering, symbol R
- added R50: 1kR, Resistors_SMD:R_0805_HandSoldering, symbol R
- added R51: R, Resistors_SMD:R_0805_HandSoldering, symbol R
- added U2: LM7805CT, TO_SOT_Packages_THT:TO-220_Neutral123_Horizontal_LargePads, symbol LM7805CT
- J1: footprint Connect:DB9FC -> Pin_Headers:Pin_Header_Straight_2x05
- U3: footprint addlol:arduino_nano -> (none)
- renumbered P2 to P2a1, P3 to P2b1, P4 to P3a1, P5 to P3b1
Connections:
- wire segments 187 -> 194
- no-connect marks 25 -> 27
Other:
- moved on the sheet: J1, P2a1

Commit message: adding stuff
Parts:
- removed P2a1, P2b1, P3a1, P3b1: CONN_02X05, Pin_Headers:Pin_Header_Straight_2x05, symbol CONN_02X05
- added C?: 100n, Capacitors_SMD:C_0805_HandSoldering, symbol C
- added P2, P4: CONN_01X05, Socket_Strips:Socket_Strip_Straight_1x05, symbol CONN_01X05
- added P3, P5: CONN_01X05, Pin_Headers:Pin_Header_Straight_1x05, symbol CONN_01X05
- added P6: CONN_01X02, Socket_Strips:Socket_Strip_Straight_1x02, symbol CONN_01X02
- C6: value C -> 100n
- R13, R14, R15, R16, R17, R18, R19, R20, R21, R22, R23, R24, R25, R26, R27, R28, R29, R30, R31, R32, R33, R34, R35, R36, R37, R39, R41, R42, R43, R44, R46, R47: value 560 -> 330
- R8: value 1kR -> 10k
Connections:
- net 12Vraw is gone; now on net 12vraw: J1.9 (P9), R3.2
- net 12vraw: no longer D13.2 (A), Q1.3 (E)
- net D4: now also P3.1 (P1)
- net D5: now also P3.2 (P2)
- net D6: now also P3.3 (P3)
- net D7: now also P3.4 (P4)
- net D8: now also P3.5 (P5)
- net GNDREF: now also J1.7 (P7), J1.8 (P8), C?.2, P4.4 (P4), P4.5 (P5), P5.4 (P4), P5.5 (P5), P6.2 (P2); no longer J1.5, R11.2
- net RST: now also C?.1
- net Vcc: now also C1.1, R11.1, P4.1 (P1), P5.1 (P1); no longer AFF1.3 (C.A.), U3.2 (3V3)
- net extShiftLight: now also P6.1 (P1); no longer J1.8 (P8)
- net gearDown: now also D10.1 (K), J1.2; no longer D10.2 (A), J1.3
- net gearUp: now also D9.1 (K), J1.4; no longer D9.2 (A), J1.2
- net intShiftLight: now also P4.3 (P3), P5.3 (P3)
- net neutral: now also D11.1 (K), J1.3; no longer D11.2 (A), J1.4
- net oilP: no longer J1.6 (P6)
- net rx: no longer U1.15 (RS232)
- net tx: no longer U1.14 (RTS)
- net 12vF: now reaches D3.2 (A), R3.1
- net 12vF: now also D13.2 (A), Q1.3 (E), P4.2 (P2), P5.2 (P2)
- net at R51.1: now also P2.1 (P1)
- net at R50.1: now also P2.5 (P5)
- net at R52.1: now also P2.2 (P2)
- net at R53.1: now also P2.3 (P3)
- net at R49.1: now also P2.4 (P4)
- removed net A6: H1.7, IC1.19 (ADC6), U3.10 (A6)
- new net: D10.2 (A), D11.2 (A), D9.2 (A), R10.1, R11.2
- no-connect marks 27 -> 36
Other:
- moved on the sheet: J1, R11

Commit message: committing very old unsaved changes
Parts:
- added SW?: REED, symbol SPST
- C3: value C -> 100n
- R1: value 2k2 -> 1k
Connections:
- net A1: now also SW?.1
- net GNDREF: now also SW?.2
Changed lines of the file:
@@
 LIBS:arduino
 LIBS:crystal_smd
+LIBS:74xgxx
+LIBS:ac-dc
+LIBS:actel
+LIBS:Altera
+LIBS:analog_devices
+LIBS:bbd
+LIBS:brooktre
+LIBS:cmos_ieee
+LIBS:dc-dc
+LIBS:diode
+LIBS:elec-unifil
+LIBS:ESD_Protection
+LIBS:ftdi
+LIBS:gennum
+LIBS:graphic
+LIBS:hc11
+LIBS:ir
+LIBS:Lattice
+LIBS:logo
+LIBS:maxim
+LIBS:microchip_dspic33dsc
+LIBS:microchip_pic10mcu
+LIBS:microchip_pic12mcu
+LIBS:microchip_pic16mcu
+LIBS:microchip_pic18mcu
+LIBS:microchip_pic32mcu
+LIBS:motor_drivers
+LIBS:msp430
+LIBS:nordicsemi
+LIBS:nxp_armmcu
+LIBS:onsemi
+LIBS:Oscillators
+LIBS:Power_Management
+LIBS:powerint
+LIBS:pspice
+LIBS:references
+LIBS:relays
+LIBS:rfcom
+LIBS:sensors
+LIBS:silabs
+LIBS:stm8
+LIBS:stm32
+LIBS:supertex
+LIBS:switches
+LIBS:transf
+LIBS:ttl_ieee
+LIBS:video
+LIBS:Worldsemi
+LIBS:Xicor
+LIBS:Zilog
 LIBS:bargraph-cache
 EELAYER 25 0
@@
 P 4000 700
 F 0 "R1" V 4080 700 50  0000 C CNN
-F 1 "2k2" V 4000 700 50  0000 C CNN
+F 1 "1k" V 4000 700 50  0000 C CNN
 F 2 "Resistors_SMD:R_0805_HandSoldering" V 3930 700 50  0001 C CNN
 F 3 "" H 4000 700 50  0000 C CNN
@@
 P 4300 900
 F 0 "C3" H 4186 946 50  0000 R CNN
-F 1 "C" H 4186 855 50  0000 R CNN
+F 1 "100n" H 4186 855 50  0000 R CNN
 F 2 "Capacitors_SMD:C_0805_HandSoldering" H 4338 750 50  0001 C CNN
 F 3 "" H 4300 900 50  0000 C CNN
@@
 	1    0    0    -1
 $EndComp
+$Comp
+L SPST SW?
+U 1 1 575C2CF3
+P 3500 4350
+F 0 "SW?" H 3500 4615 50  0000 C CNN
+F 1 "REED" H 3500 4524 50  0000 C CNN
+F 2 "" H 3500 4350 50  0000 C CNN
+F 3 "" H 3500 4350 50  0000 C CNN
+	1    3500 4350
+	1    0    0    -1
+$EndComp
+$Comp
+L GNDREF #PWR?
+U 1 1 575C3B39
+P 4000 4350
+F 0 "#PWR?" H 4000 4100 50  0001 C CNN
+F 1 "GNDREF" H 4000 4200 50  0001 C CNN
+F 2 "" H 4000 4350 50  0000 C CNN
+F 3 "" H 4000 4350 50  0000 C CNN
+	1    4000 4350
+	1    0    0    -1
+$EndComp
+Text Label 3000 4350 2    60   ~ 0
+A1
 $EndSCHEMATC
